File: hardware/usb-sniffer.kicad_sch (KiCad schematic)
At the start: 40 parts, among them IC1 LCMXO2-2000HC, IC2 MIC5504-3.3v, J1 USB-C, J2 USB-C, J3 USB-A, J4 IN, J5 GND

Commit message: Use a single large sheet for the schematic
Parts:
- removed J1, J2: USB-C, ataradov_conn:USB-C, symbol ataradov_conn:USB-C
- removed J3: USB-A, ataradov_conn:USB-A-Slots, symbol ataradov_conn:USB-A
- added C11, C12, C13, C16, C17, C18, C19, C20, C22, C23, C24, C25, C26, C27, C28, C29: 100nF, ataradov_smd:0603, symbol ataradov_rlc:C
- added C14, C15, C30, C31: 2.2uF, ataradov_smd:0603, symbol ataradov_rlc:C
- added C21: 10uF, ataradov_smd:0603, symbol ataradov_rlc:C
- added IC10: DSC6101CI2A-024.0000, ataradov_ic:CDFN-4-3.2x2.5mm, symbol ataradov_crystal:DSC61XX-MHz
- added IC3, IC5, IC7: MAX9032AKA+T, ataradov_ic:SOT-23-8, symbol ataradov_ic:Comp-Dual
- added IC4: USB3343, ataradov_ic:QFN-24-0.5mm, symbol ataradov_ic:USB3343
- added IC6: DSC6101CI2A-026.0000, ataradov_ic:CDFN-4-3.2x2.5mm, symbol ataradov_crystal:DSC61XX-MHz
- added IC8: I2C-EEPROM, ataradov_ic:SO-8, symbol ataradov_ic:I2C-EEPROM
- added IC9: CY7C68013A-56PVXC, ataradov_ic:SSOP-56-0.635mm, symbol ataradov_mcu:CY7C68013A-56PVXC
- added J1: CONTROL, symbol Connector:USB_C_Receptacle_USB2.0
- added J2: HOST, symbol Connector:USB_C_Receptacle_USB2.0
- added J3: TEST_DEVICE, symbol Connector:USB_A
- added LED7: Yellow, ataradov_smd:0603, symbol ataradov_led:LED
- added R10: 20K, ataradov_smd:0603, symbol ataradov_rlc:R
- added R11: 8.06K, ataradov_smd:0603, symbol ataradov_rlc:R
- added R12, R13, R18, R19, R21: 10K, ataradov_smd:0603, symbol ataradov_rlc:R
- added R14: 33K, ataradov_smd:0603, symbol ataradov_rlc:R
- added R15, R16: 4.7K, ataradov_smd:0603, symbol ataradov_rlc:R
- added R17, R20: 100, ataradov_smd:0603, symbol ataradov_rlc:R
- added RN2: 2.2K, ataradov_smd:0603x4, symbol ataradov_rlc:RN-4
- added TP10: BOOT, ataradov_misc:TestPoint-1.27mm, symbol ataradov_misc:TestPoint
- added TP11: RESET, ataradov_misc:TestPoint-1.27mm, symbol ataradov_misc:TestPoint
- added TP12: GND, ataradov_misc:TestPoint-1.27mm, symbol ataradov_misc:TestPoint
- added TP9: VCC, ataradov_misc:TestPoint-1.27mm, symbol ataradov_misc:TestPoint
Connections:
- net +3V3: now also C11.2, C12.2, C13.2, C16.2, C17.2, C18.2, C19.2, C20.2, C22.2, C23.2, C24.2, C25.2, C26.2, C27.2, C28.2, C29.2, C30.2, C31.2, IC10.1 (OE), IC10.4 (VCC), IC3.8 (VCC), IC4.16 (VBAT), IC4.9 (VDDIO), IC5.8 (VCC), IC6.1 (OE), IC6.4 (VCC), IC7.8 (VCC), IC8.1 (A0), IC8.8 (VCC), IC9.10 (AVCC*2), IC9.14 (AVCC), IC9.18 (VCC), IC9.24 (VCC), IC9.34 (VCC), IC9.39 (VCC), IC9.50 (VCC), IC9.6 (VCC*6), R12.2, R13.2, R19.1, R21.2, RN2.7, RN2.8, TP9.1
- net CMP_DM_1: now also IC3.1
- net CMP_DM_2: now also IC5.1
- net CMP_DM_3: now also IC7.1
- net CMP_DP_1: now also IC3.7
- net CMP_DP_2: now also IC5.7
- net CMP_DP_3: now also IC7.7
- net CTRL_CLK: now also IC9.40 (PA0/~{INT0})
- net CTRL_DATA: now also IC9.43 (PA3/WU2)
- net FD0: now also IC9.25 (PB0/FD0)
- net FD1: now also IC9.26 (PB1/FD1)
- net FD10: now also IC9.54 (PD2/FD10)
- net FD11: now also IC9.55 (PD3/FD11)
- net FD12: now also IC9.56 (PD4/FD12)
- net FD13: now also IC9.1 (PD5/FD13)
- net FD14: now also IC9.2 (PD6/FD14)
- net FD15: now also IC9.3 (PD7/FD15)
- net FD2: now also IC9.27 (PB2/FD2)
- net FD3: now also IC9.28 (PB3/FD3)
- net FD4: now also IC9.29 (PB4/FD4)
- net FD5: now also IC9.30 (PB5/FD5)
- net FD6: now also IC9.31 (PB6/FD6)
- net FD7: now also IC9.32 (PB7/FD7)
- net FD8: now also IC9.52 (PD0/FD8)
- net FD9: now also IC9.53 (PD1/FD9)
- net FLAGA: now also IC9.36 (CTL0/FLAGA)
- net FLAGB: now also IC9.37 (CTL1/FLAGB)
- net FLAGC: now also IC9.38 (CTL2/FLAGC)
- net FOFOADR0: now also IC9.44 (PA4/FIFOADR0)
- net FOFOADR1: now also IC9.45 (PA5/FIFOADR1)
- net GPIO: now also IC9.47 (PA7/FLAGD/~{SLCS})
- net IFCLK: now also IC9.20 (IFCLK/T0OUT)
- net JTAGEN: now also IC9.41 (PA1/~{INT1})
- net PKTEND: now also IC9.46 (PA6/PKTEND)
- net SLOE: now also IC9.42 (PA2/SLOE)
- net SLRD: now also IC9.8 (RDY0/SLRD)
- net SLWR: now also IC9.9 (RDY1/SLWR)
- net T_USB_CLK: now also IC4.2 (CLKOUT)
- net T_USB_D0: now also IC4.4 (D0)
- net T_USB_D1: now also IC4.5 (D1)
- net T_USB_D2: now also IC4.6 (D2)
- net T_USB_D3: now also IC4.7 (D3)
- net T_USB_D4: now also IC4.8 (D4)
- net T_USB_D5: now also IC4.10 (D5)
- net T_USB_D6: now also IC4.11 (D6)
- net T_USB_D7: now also IC4.12 (D7)
- net T_USB_DIR: now also IC4.1 (DIR)
- net T_USB_NXT: now also IC4.3 (NXT)
- net T_USB_STP: now also IC4.24 (STP)
- net at R4.2: now also J2.B5 (CC2)
- net at R5.2: now also J2.A5 (CC1)
- net at R1.2: now also J1.B5 (CC2)
- net at R2.2: now also J1.A5 (CC1)
- net GND renamed AGND
- net AGND: now also C11.1, C12.1, C13.1, C14.1, C15.1, C16.1, C17.1, C18.1, C19.1, C20.1, C21.1, C22.1, C23.1, C24.1, C25.1, C26.1, C27.1, C28.1, C29.1, C30.1, C31.1, IC10.2 (GND), IC3.4 (GND), IC4.25 (PAD), IC5.4 (GND), IC6.2 (GND), IC7.4 (GND), IC8.3 (A2), IC8.4 (GND), IC8.7 (WP), IC9.13 (AGND*2), IC9.17 (AGND), IC9.19 (GND), IC9.21 (RSVD), IC9.33 (GND), IC9.35 (GND), IC9.4 (GND*6), IC9.48 (GND), IC9.7 (GND), J1.A1 (GND), J1.A12 (GND), J1.B1 (GND), J1.B12 (GND), J1.S1 (SHIELD), J2.A1 (GND), J2.A12 (GND), J2.B1 (GND), J2.B12 (GND), J2.S1 (SHIELD), J3.4 (GND), J3.5 (Shield), LED7.2 (K), R11.1, R16.1, RN2.5, RN2.6, TP12.1
- new net: C14.2, IC4.15 (VDD33), IC4.18 (ID)
- new net: LED7.1 (A), R18.1
- new net: J2.A4 (VBUS), J2.A9 (VBUS), J2.B4 (VBUS), J2.B9 (VBUS), J3.1 (VBUS), R10.2, R18.2
- new net: C15.2, IC4.23 (VDD18)
- new net: IC9.51 (WAKEUP), R19.2
- new net: IC4.22 (RESETB), R13.1
- new net: IC4.17 (VBUS), R10.1
- new net: IC10.3 (OUT), R20.1
- new net: J1.A4 (VBUS), J1.A9 (VBUS), J1.B4 (VBUS), J1.B9 (VBUS)
- new net: IC9.15 (DPLUS), J1.A6 (D+), J1.B6 (D+)
- new net: IC9.16 (DMINUS), J1.A7 (D-), J1.B7 (D-)
- new net: IC4.19 (RBIAS), R11.2
- new net: IC6.3 (OUT), R17.1
- new net A1: IC8.2 (A1), RN2.3, RN2.4, TP10.1
- new net CMP_REF_1: IC3.2 (-), IC3.6 (-), R15.1, R16.2
- new net CMP_REF_2: IC5.2 (-), IC5.6 (-), R14.1, R15.2
- new net CMP_REF_3: IC7.2 (-), IC7.6 (-), R12.1, R14.2
- new net CY_CLK: IC9.12 (XTALIN), R20.2
- new net RESET: C21.2, IC9.49 (~{RESET}), R21.1, TP11.1
- new net SCL: IC8.6 (SCL), IC9.22 (SCL), RN2.2
- new net SDA: IC8.5 (SDA), IC9.23 (SDA), RN2.1
- new net T_USB_D+: IC3.5 (+), IC4.14 (DM), IC5.5 (+), IC7.5 (+), J2.A6 (D+), J2.B6 (D+), J3.3 (D+)
- new net T_USB_D-: IC3.3 (+), IC4.13 (DP), IC5.3 (+), IC7.3 (+), J2.A7 (D-), J2.B7 (D-), J3.2 (D-)
- new net USB_CLK_IN: IC4.21 (XI), R17.2
- no-connect marks 0 -> 20
Other:
- removed sheet Host USB
- removed sheet Target USB
- note removed: "USB Sniffer v6"
- moved on the sheet: C1, C10, C2, C3, C4, C5, C6, C7, C8, C9, D1, IC1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
